File: Kicad/OpenReflowPlate/OpenReflowPlate.kicad_sch (KiCad schematic)
At the start: 19 parts, among them IC2 MAX31855KASA+, U1 STM32L476RGTx

Commit message: last version
Parts:
- added C1, C2: 100nF, CAPC2012X140N, symbol Library_Loader:C0805C475M8RACTU
- added C_22p_? (x4): 22pF, User_lib:CAPC2012X140N, symbol PicBytesMicro-rescue:GCG21BR71H154KA01K-SamacSys_Parts
- added D1, D2: ZLLS410TA, SOD2513X120N, symbol User_lib:ZLLS410TA
- added IC1: TC1108-3.3VDBTR, SOT230P700X180-4N, symbol Library_Loader:TC1108-3.3VDBTR
- added J1: TC connector, 282834-2_1, symbol Library_Loader:282834-2
- added J2: Type - C, 2169900003, symbol Library_Loader:216990-0003
- added J2: B2B-XH-A, B2BXHA, symbol User_lib:B2B-XH-A
- added J3: Output_AC, 691411910003, symbol SMPS-rescue:691411910003-691411910003
- added J4: Input_AC, 691411910003, symbol SMPS-rescue:691411910003-691411910003
- added J6: TC2030-MCP-NL, TC2030-MCP-NL, symbol User_lib:TC2030-MCP-NL
- added K1: SSRC-240D5R, SSRC240D5R, symbol User_lib:SSRC-240D5R
- added K2: HF49FD_012-1H12F, HF49FD0121H12F, symbol User_lib:HF49FD_012-1H12F
- added LS1: TMB12A05, TMB12A05, symbol User_lib:TMB12A05
- added PS1: HLK-PM03, HLKPM03, symbol User_lib:HLK-PM03
- added Q1, Q2, Q3, Q4, Q5 (x3): SMMBT5551LT1G, SOT96P237X111-3N, symbol BytesCounter-rescue:SMMBT5551LT1G-SamacSys_Parts
- added R1, R13 (x3), R5, R7, R9: 4k7, RESC2012X65N, symbol BytesCounter-rescue:KTR10EZPF4220-SamacSys_Parts
- added R10, R4, R6, R8: 100, RESC2012X65N, symbol BytesCounter-rescue:KTR10EZPF4220-SamacSys_Parts
- added R13: 0, Resistor_SMD:R_0805_2012Metric, symbol OpenReflowPlate-rescue:ERJP6WF1303V-Library_Loader
- added R14: 220, RESC2012X65N, symbol BytesCounter-rescue:KTR10EZPF4220-SamacSys_Parts
- added R_10K_2, R_10K_4, R_10K_5: 10k, User_lib:RESC2012X75N, symbol PicBytesMicro-rescue:KTR10EZPF4220-SamacSys_Parts
- added R_10K_3, R_10K_7, R_10K_9: 10k, RESC2012X65N, symbol PicBytesMicro-rescue:KTR10EZPF4220-SamacSys_Parts
- added R_10K_6: 10K, RESC2012X65N, symbol PicBytesMicro-rescue:KTR10EZPF4220-SamacSys_Parts
- added R_10K_8: 10K, User_lib:RESC2012X75N, symbol PicBytesMicro-rescue:KTR10EZPF4220-SamacSys_Parts
- added S_down1: Back Button, 430182070816, symbol User_lib:430182050816
- added S_left1: Right Button, 430182070816, symbol User_lib:430182050816
- added S_right1: Enter Button, 430182070816, symbol User_lib:430182050816
- added S_up1: Left Button, 430182070816, symbol User_lib:430182050816
- added U1: CC56-12EWA, Display_7Segment:CA56-12EWA, symbol Display_Character:CC56-12EWA
- R2: value 220 -> 1k
- renumbered C1 to C4, C2 to C5, C3 to C6, C4 to C7, LED2 to LED1, LED1 to LED2, R1 to R14, R3 to R4, R4 to R7, R5 to R8, U1 to U2
Connections:
- net +3V3: now also C2.1, IC1.3 (VOUT), J6.1 (-MCLR/VPP), R_10K_3.2, R_10K_5.2, R_10K_7.2, R_10K_9.2; no longer LED4.2
- net GND: now also C1.2, C2.2, C_22p_?.1, C_22p_?.2, C_22p_?.2, C_22p_?.2, IC1.2 (GND_1), IC1.4 (GND_2), J2.1, J2.A1 (GND_1), J2.A12 (GND_2), J2.MH1, J2.MH2, J2.MH3, J2.MH4, J6.5 (PGC_(ICSPCLK)), K1.4 (_-DC_INPUT), K2.4 (COIL_2), LS1.2 (-), PS1.3 (-V0), Q1.2, Q2.2, Q3.2, Q4.2, S_down1.2, S_down1.4, S_left1.2, S_left1.4, S_right1.2, S_right1.4, S_up1.2, S_up1.4
- net LED_OUT1: now also U2.8 (PC0); no longer U2.26 (PB0)
- net LED_OUT2: now also U2.9 (PC1); no longer U2.27 (PB1)
- net SWCLK: now also J6.4 (PGD_(ICSPDAT))
- net SWDIO: now also J6.2 (VDD)
- net USB_D+: now also J2.A6 (DP1), J2.B6 (DP2)
- net USB_D-: now also J2.A7 (DN1), J2.B7 (DN2)
- net LED_LIFE: now reaches U2.10 (PC2)
- net LED_LIFE: now also LED4.2
- net at U2.2 (PC13): now also R13.1
- net C_3: now reaches U2.28 (PB2)
- net C_3: now also R7.1
- net D_g: now reaches U2.29 (PB10)
- net D_g: now also U1.5 (g)
- net D_dp: now reaches U2.30 (PB11)
- net D_dp: now also U1.3 (DPX)
- net C_buzzer: now reaches U2.34 (PB13)
- net C_buzzer: now also R13.1
- net C_out1: now reaches U2.35 (PB14)
- net C_out1: now also R13.1
- net C_out2: now reaches U2.36 (PB15)
- net C_out2: now also R13.1
- net BUT_LEFT: now reaches U2.40 (PC9)
- net BUT_LEFT: now also C_22p_?.2, R_10K_6.2
- net BUT_RIGHT: now reaches U2.51 (PC10)
- net BUT_RIGHT: now also C_22p_?.1, R_10K_2.1
- net BUT_ENTER: now reaches U2.52 (PC11)
- net BUT_ENTER: now also C_22p_?.1, R_10K_8.1
- net BUT_BACK: now reaches U2.53 (PC12)
- net BUT_BACK: now also C_22p_?.1, R_10K_4.1
- net C_4: now reaches U2.55 (PB3)
- net C_4: now also R9.1
- net D_a: now reaches U2.56 (PB4)
- net D_a: now also U1.11 (a)
- net D_b: now reaches U2.57 (PB5)
- net D_b: now also U1.7 (b)
- net D_c: now reaches U2.58 (PB6)
- net D_c: now also U1.4 (c)
- net D_d: now reaches U2.59 (PB7)
- net D_d: now also U1.2 (d)
- net D_e: now reaches U2.61 (PB8)
- net D_e: now also U1.1 (e)
- net D_f: now reaches U2.62 (PB9)
- net D_f: now also U1.10 (f)
- net reset: now reaches U2.7 (NRST)
- net reset: now also J6.3 (GND)
- net LED_AC renamed AC_Vdcin+
- net AC_Vdcin+: now also D2.2, K2.2 (NO), PS1.4 (+V0), R13.2
- net T+_tcm1: no longer names the net of LFB1.1
- net T+_tcm1: now also J1.1
- net T-_tcm1: no longer names the net of LFB2.1
- net T-_tcm1: now also J1.2
- new net: J3.1, J3.A1, K1.2 (AC_LOAD_2)
- new net: Q5.1, R13.2 (x3)
- new net: R_10K_2.2, R_10K_3.1, S_left1.1, S_left1.3
- new net: R_10K_8.2, R_10K_9.1, S_right1.1, S_right1.3
- new net: Q1.1, R1.2
- new net: Q1.3, R4.1
- new net: R_10K_5.1, R_10K_6.1, S_up1.1, S_up1.3
- new net: Q3.1, R7.2
- new net: Q4.3, R10.1
- new net: Q2.3, R6.1
- new net: Q3.3, R8.1
- new net: Q5.3, R14.2
- new net: Q2.1, R5.2
- new net: LS1.1 (+), Q5.2
- new net: R_10K_4.2, R_10K_7.1, S_down1.1, S_down1.3
- new net: Q4.1, R9.2
- new net +5V: C1.1, D1.1, D2.1, IC1.1 (VIN), Q5.3, Q5.3, R14.1
- new net AC_L: J4.1, J4.A1, K1.1 (AC_LOAD_1), PS1.1 (AC_1)
- new net AC_N: J3.2, J3.A2, J4.2, J4.A2, PS1.2 (AC_2)
- new net AC_ground: J3.3, J3.A3, J4.3, J4.A3
- new net Activation_out1: K1.3 (+DC_INPUT), Q5.2
- new net Activation_out2: K2.3 (COIL_1), Q5.2
- new net CC_1: R4.2, U1.12 (CC1)
- new net CC_2: R6.2, U1.9 (CC2)
- new net CC_3: R8.2, U1.8 (CC3)
- new net CC_4: R10.2, U1.6 (CC4)
- new net C_1: R1.1, U2.26 (PB0)
- new net C_2: R5.1, U2.27 (PB1)
- new net DC_Out2: J2.2, K2.1 (COM)
- new net USB_Vin+: D1.2, J2.A4 (VBUS_1), J2.A9 (VBUS_2)
- no-connect marks 4 -> 27
Other:
- note added: "AC Output // Output 1"
- note added: "AC input / HILINK Converter ACDC"
- note added: "Buttons Circuity"
- note added: "Buzzer"
- note added: "DC Output // Output 2"
- note added: "Display"
- note added: "For ST32 and ARM CORTEX SWD: 1-VCC 2-SWDIO / TMS 3-nRESET 4-SWCLK / TCK 5 GND 6 SWO / TDO"
- note added: "Output1"
- note added: "Output2"
- note added: "Outputs of the system -Output1: AC Relay -Output2: DC Relay"
- note added: "Programming port using TAG-CONNECT to ST32"
- note added: "STM32L476RG Microcontroller"
- note added: "USB type C Entry"
- note added: "Voltage Regulator 5V to 3.3V Both entries are possible: USB or AC"
- moved on the sheet: C4, C5, C6, C7, JP1, LED1, LED2, LED3, LED4, R14, R2, R4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

Commit message: V1 HW
Parts:
- removed J2: Type - C, 2169900003, symbol Library_Loader:216990-0003
- removed K2: HF49FD_012-1H12F, HF49FD0121H12F, symbol User_lib:HF49FD_012-1H12F
- removed PS1: HLK-PM03, HLKPM03, symbol User_lib:HLK-PM03
- added J7: 629722000214, usb-c:629722000214, symbol usb-type-c:629722000214
- added K3: HF49FD_012-1H11F, HF49FD0121H11F, symbol User:HF49FD_012-1H11F
- added PS2: HLK-5M05, HLK5M05, symbol User:HLK-5M05
Connections:
- net AC_L: now also PS2.1 (AC_1)
- net AC_N: now also PS2.2 (AC_2)
- net AC_Vdcin+: now also K3.2 (NO), PS2.4 (+VO)
- net Activation_out2: now also K3.3 (COIL_1)
- net DC_Out2: now also K3.1 (COM)
- net GND: now also J7.A1 (GND), J7.A12 (GND1), J7.B1 (GND3), J7.B12 (GND2), J7.S1, J7.S2, J7.S3, J7.S4, K3.4 (COIL_2), PS2.3 (-VO)
- net USB_D+: now also J7.A6 (D+1), J7.B6 (D+2)
- net USB_D-: now also J7.A7 (D-1), J7.B7 (D-2)
- net USB_Vin+: now also J7.A4 (VBUS), J7.A9 (VBUS1), J7.B4 (VBUS3), J7.B9 (VBUS2)
Other:
- note added: "**CHANGELOG** *****V1***** -Changed HF49-12 to HF49-11 footprint. -Fix HI-LINK footprint -Fix Display footprint -Fix enter button -Improved USB communication lines -New USB type C"
